Commit message: modify robot.urdf for sapien 2

File: ace_teleop/dynamixel/urdf/left_arm/robot.urdf (robot description, URDF)
Before this commit: robot onshape, 8 links, 7 joints
Links:
- link base: mass 0.58379058258406058002 -> 0.583
- link connection: mass 0.083862510289046426903 -> 0.083
- link ee_c: mass 0.00098125000000000013427 -> 0
- link forearm_left: mass 1.3817156104582399845 -> 1.381
- link link_0: mass 0.17595724897368519857 -> 0.175
- link link_1: mass 0.17595724897368519857 -> 0.175
- link upperarm: mass 1.0941679996560738086 -> 1.094
- link wrist: mass 0.6581458956762692436 -> 0.658
Joints:
- joint 1: limit lower=-1.570796326794896558 upper=1.570796326794896558 effort=1 velocity=20 -> lower=-1.57 upper=1.57 effort=1 velocity=20; origin xyz=-0.015300000000000084366 -2.7755575615628913511e-17 0.054999999999998952505 rpy=-1.570796326794896336 3.1918911957973087835e-16 -1.5707963267948970021 -> xyz=-0.015 0 0.054 rpy=-1.57 0 -1.57
- joint 2: limit lower=-1.570796326794896558 upper=1.2217304763960306069 effort=1 velocity=20 -> lower=-1.57 upper=1.221 effort=1 velocity=20; origin xyz=-1.0394463068053101868e-15 -0.29999999999999815703 5.9188765000328658061e-15 rpy=-3.1415926535897908956 -2.5975450053993224616e-15 -1.493953510915167858e-14 -> xyz=0 -0.299 0 rpy=-3.141 0 0
- joint 3: limit lower=-0.785398163397448279 upper=1.570796326794896558 effort=1 velocity=20 -> lower=-0.785 upper=1.57 effort=1 velocity=20; origin xyz=-0.0074000000000039494255 0.017750000000001708855 -0.015299999999999654154 rpy=1.570796326794926534 -1.5707963267948692465 0 -> xyz=-0.007 0.017 -0.015 rpy=1.57 -1.57 0
- joint 4: limit lower=-1.570796326794896558 upper=1.570796326794896558 effort=1 velocity=20 -> lower=-1.57 upper=1.57 effort=1 velocity=20; origin xyz=2.6386656104519486103e-16 0.025500000000000050404 0.020500000000000018208 rpy=1.57079632679489678 -0.011253197791822201063 -1.0282839359771659263e-14 -> xyz=0 0.025 0.02 rpy=1.57 -0.011 0
- joint 5: limit lower=-1.2217304763960306069 upper=1.2217304763960306069 effort=1 velocity=20 -> lower=-1.221 upper=1.221 effort=1 velocity=20; origin xyz=-0.018500000000011597445 -0.0074000000000039589665 -0.31120000000001674101 rpy=-3.7339808647203377508e-14 1.5707963267947984143 0 -> xyz=-0.018 -0.007 -0.311 rpy=0 1.57 0
- joint 6: limit lower=-1.570796326794896558 upper=1.570796326794896558 effort=1 velocity=20 -> lower=-1.57 upper=1.57 effort=1 velocity=20; origin xyz=0.007600000000057283156 0.0177500000000477276 -0.01529999999996361007 rpy=1.5707963267949778263 -1.5707963267948557018 0 -> xyz=0.007 0.017 -0.015 rpy=1.57 -1.57 0
- joint ee: origin xyz=1.1796119636642288242e-15 -0.12399999999999949951 -0.074499999999995403233 rpy=-1.5707963267949078823 -2.8813146539454304284e-17 -1.5707963267949036634 -> xyz=0 -0.123 -0.074 rpy=-1.57 0 -1.57

File: ace_teleop/dynamixel/urdf/left_arm_m/robot.urdf (robot description, URDF)
Before this commit: robot onshape, 8 links, 7 joints
Links:
- link base: mass 0.58379058258406058002 -> 0.583
- link connection: mass 0.083862510289046426903 -> 0.083
- link ee_c: mass 0.00098125000000000013427 -> 0
- link forearm_left: mass 1.3817156104582399845 -> 1.381
- link link_0: mass 0.17595724897368519857 -> 0.175
- link link_1: mass 0.17595724897368519857 -> 0.175
- link upperarm: mass 1.0941679996560738086 -> 1.094
- link wrist: mass 0.6581458956762692436 -> 0.658
Joints:
- joint 1: limit lower=-3.141592653589793116 upper=1.570796326794896558 effort=1 velocity=20 -> lower=-3.141 upper=1.57 effort=1 velocity=20; origin xyz=-0.0039599313900715304992 -0.055000000000002685629 -0.014778665142207866867 rpy=-2.836498295494452124e-13 0.26179938779907696578 -1.4109997389838678056e-13 -> xyz=-0.003 -0.055 -0.014 rpy=0 0.261 0
- joint 2: limit lower=-1.570796326794896558 upper=1.570796326794896558 effort=1 velocity=20 -> lower=-1.57 upper=1.57 effort=1 velocity=20; origin xyz=-1.6245844983992342151e-13 -0.30000000000024223956 -1.108661773496777414e-14 rpy=3.1415926535895084548 -7.2845193525401583906e-14 -9.2134271856746957148e-14 -> xyz=0 -0.3 0 rpy=3.141 0 0
- joint 3: limit lower=-1.570796326794896558 upper=1.570796326794896558 effort=1 velocity=20 -> lower=-1.57 upper=1.57 effort=1 velocity=20; origin xyz=-0.0074000000000020351582 0.01775000000000098721 -0.01530000000000937381 rpy=1.570796326794911435 -1.5707963267948541475 0 -> xyz=-0.007 0.017 -0.015 rpy=1.57 -1.57 0
- joint 4: limit lower=-4.712388980384689674 upper=1.570796326794896558 effort=1 velocity=20 -> lower=-4.712 upper=1.57 effort=1 velocity=20; origin xyz=2.6855733172047512218e-16 0.02550000000000007469 0.020499999999999851674 rpy=1.570796326794896558 -0.011253197791837232442 -1.0675177281981156857e-14 -> xyz=0 0.025 0.02 rpy=1.57 -0.011 0
- joint 5: limit lower=-1.570796326794896558 upper=1.570796326794896558 effort=1 velocity=20 -> lower=-1.57 upper=1.57 effort=1 velocity=20; origin xyz=-0.018500000000000061534 -0.0073999999999964094499 -0.31120000000003522622 rpy=-1.5707963267949236474 1.5656486849775397285 -1.5707963267936464469 -> xyz=-0.018 -0.007 -0.311 rpy=-1.57 1.565 -1.57
- joint 6: limit lower=-1.570796326794896558 upper=1.570796326794896558 effort=1 velocity=20 -> lower=-1.57 upper=1.57 effort=1 velocity=20; origin xyz=0.0076000000000781553489 0.017750000000072096995 -0.015299999999993540989 rpy=1.5707963223908167905 -1.5707878466134952422 3.568907028788945584e-09 -> xyz=0.007 0.017 -0.015 rpy=1.57 -1.57 0
- joint ee: origin xyz=1.1865508575681360526e-15 -0.12399999999999961053 -0.074499999999995403233 rpy=-1.5707963267949078823 -2.6347357475703645387e-17 -1.570796326794896336 -> xyz=0 -0.123 -0.074 rpy=-1.57 0 -1.57

File: ace_teleop/dynamixel/urdf/right_arm/robot.urdf (robot description, URDF)
Before this commit: robot onshape, 8 links, 7 joints
Links:
- link base: mass 0.58379058258406058002 -> 0.583
- link connection: mass 0.083862510289046426903 -> 0.083
- link ee_c: mass 0.00098125000000000013427 -> 0
- link forearm_right: mass 1.3817156104582397624 -> 1.381
- link link_0: mass 0.17595724897368519857 -> 0.175
- link link_1: mass 0.17595724897368519857 -> 0.175
- link upperarm: mass 1.0941679996560738086 -> 1.094
- link wrist: mass 0.6581458956762692436 -> 0.658
Joints:
- joint 1: limit lower=-1.570796326794896558 upper=1.570796326794896558 effort=1 velocity=20 -> lower=-1.57 upper=1.57 effort=1 velocity=20; origin xyz=0.015299999999999957731 -1.2143064331837649661e-16 0.054999999999998883116 rpy=-1.570796326794896336 -3.1918911957972432094e-16 1.5707963267948972241 -> xyz=0.015 0 0.054 rpy=-1.57 0 1.57
- joint 2: limit lower=-1.2217304763960306069 upper=1.570796326794896558 effort=1 velocity=20 -> lower=-1.221 upper=1.57 effort=1 velocity=20; origin xyz=-1.5869250358235869954e-15 -0.29999999999999871214 -3.3827107781547738341e-16 rpy=-3.141592653589793116 6.6613381477543983976e-16 -5.7511253411613382311e-15 -> xyz=0 -0.299 0 rpy=-3.141 0 0
- joint 3: limit lower=-1.570796326794896558 upper=0.785398163397448279 effort=1 velocity=20 -> lower=-1.57 upper=0.785 effort=1 velocity=20; origin xyz=0.0075999999999946336177 0.01774999999999710143 -0.015300000000015237175 rpy=1.5707963267947866459 1.5707963267948945596 0 -> xyz=0.007 0.017 -0.015 rpy=1.57 1.57 0
- joint 4: limit lower=-1.570796326794896558 upper=1.570796326794896558 effort=1 velocity=20 -> lower=-1.57 upper=1.57 effort=1 velocity=20; origin xyz=2.6252869104828667613e-16 0.025500000000000053874 0.020499999999999907185 rpy=1.57079632679489678 -0.011253197791837241115 -4.576144232712457471e-15 -> xyz=0 0.025 0.02 rpy=1.57 -0.011 0
- joint 5: limit lower=-1.2217304763960306069 upper=1.2217304763960306069 effort=1 velocity=20 -> lower=-1.221 upper=1.221 effort=1 velocity=20; origin xyz=0.018499999999998434363 -0.007599999999997830713 -0.31120000000000513918 rpy=-1.427545892204754887e-14 -1.5707963267948232833 0 -> xyz=0.018 -0.007 -0.311 rpy=0 -1.57 0
- joint 6: limit lower=-1.570796326794896558 upper=1.570796326794896558 effort=1 velocity=20 -> lower=-1.57 upper=1.57 effort=1 velocity=20; origin xyz=-0.0073999999999662113837 0.017750000000061827432 -0.015300000000086263693 rpy=1.5707963267948485964 1.5707963267948832353 0 -> xyz=-0.007 0.017 -0.015 rpy=1.57 1.57 0
- joint ee: origin xyz=1.1657341758564143674e-15 -0.12399999999999961053 -0.074499999999995458744 rpy=1.5707963267949078823 2.6235511861393905573e-17 1.5707963267948978903 -> xyz=0 -0.123 -0.074 rpy=1.57 0 1.57

File: ace_teleop/dynamixel/urdf/right_arm_m/robot.urdf (robot description, URDF)
Before this commit: robot onshape, 8 links, 7 joints
Links:
- link base: mass 0.58379058258406058002 -> 0.583
- link connection: mass 0.083862510289046426903 -> 0.083
- link ee_c: mass 0.00098125000000000013427 -> 0
- link forearm_right: mass 1.3817156104582397624 -> 1.381
- link link_0: mass 0.17595724897368519857 -> 0.175
- link link_1: mass 0.17595724897368519857 -> 0.175
- link upperarm: mass 1.0941679996560738086 -> 1.094
- link wrist: mass 0.6581458956762692436 -> 0.658
Joints:
- joint 1: limit lower=-1.570796326794896558 upper=3.141592653589793116 effort=1 velocity=20 -> lower=-1.57 upper=3.141 effort=1 velocity=20; origin xyz=0.0039599313900685866735 -0.054999999999998994138 -0.014778665142222695283 rpy=-1.5149872090953951554e-15 -0.26179938779915112868 1.065294583260393049e-15 -> xyz=0.003 -0.054 -0.014 rpy=0 -0.261 0
- joint 2: limit lower=-1.570796326794896558 upper=1.570796326794896558 effort=1 velocity=20 -> lower=-1.57 upper=1.57 effort=1 velocity=20; origin xyz=3.729547893732891099e-16 -0.29999999999999876765 -1.3669620990697239904e-15 rpy=-3.1415926535897917837 1.9012525540606479163e-15 -2.8053523899771700523e-15 -> xyz=0 -0.299 0 rpy=-3.141 0 0
- joint 3: limit lower=-1.570796326794896558 upper=1.570796326794896558 effort=1 velocity=20 -> lower=-1.57 upper=1.57 effort=1 velocity=20; origin xyz=0.0076000000000075867979 0.01774999999999854472 -0.015300000000058105662 rpy=1.5707963267947875341 1.5707963267944859975 0 -> xyz=0.007 0.017 -0.015 rpy=1.57 1.57 0
- joint 4: limit lower=-1.570796326794896558 upper=4.712388980384689674 effort=1 velocity=20 -> lower=-1.57 upper=4.712 effort=1 velocity=20; origin xyz=2.639854242781557983e-16 0.025500000000000060812 0.020499999999999962697 rpy=1.57079632679489678 -0.011253197791837133562 -1.0010230155453631437e-14 -> xyz=0 0.025 0.02 rpy=1.57 -0.011 0
- joint 5: limit lower=-1.570796326794896558 upper=1.570796326794896558 effort=1 velocity=20 -> lower=-1.57 upper=1.57 effort=1 velocity=20; origin xyz=0.018499999999994409805 -0.0076000000000094325436 -0.31120000000002756568 rpy=-5.4841195482422594032e-14 -1.5707963267948292785 0 -> xyz=0.018 -0.007 -0.311 rpy=0 -1.57 0
- joint 6: limit lower=-1.570796326794896558 upper=1.570796326794896558 effort=1 velocity=20 -> lower=-1.57 upper=1.57 effort=1 velocity=20; origin xyz=-0.0073999999999634913372 0.017750000000063881345 -0.01530000000009469445 rpy=1.5707963267948352737 1.570796326794886788 0 -> xyz=-0.007 0.017 -0.015 rpy=1.57 1.57 0
- joint ee: origin xyz=1.1067535776732029262e-15 -0.12399999999999966604 -0.074499999999995458744 rpy=1.5707963267949078823 2.9290282597286045162e-17 1.5707963267948970021 -> xyz=0 -0.123 -0.074 rpy=1.57 0 1.57
