Commit message: easy to understand coordinate frame definition

File: ace_teleop/assets/xarm7_ability/xarm7_ability.urdf (robot description, URDF)
Before this commit: robot xarm7_ability, 53 links, 52 joints
Links:
- link l_base: geometry collision mesh filename=../ability_hand/meshes/collision/wristmesh_C.obj; visual mesh filename=../ability_hand/meshes/visual/wristmesh.obj
- link l_index_L1: geometry collision box size=0.012 0.012 0.002; collision box size=0.012 0.012 0.002
- link l_index_L2: geometry collision mesh filename=../ability_hand/meshes/collision/idx-F2_C.obj; collision sphere radius=0.007
- link l_middle_L1: geometry collision box size=0.012 0.012 0.002; collision box size=0.012 0.012 0.002
- link l_middle_L2: geometry collision mesh filename=../ability_hand/meshes/collision/idx-F2_C.obj; collision sphere radius=0.007
- link l_pinky_L1: geometry collision box size=0.012 0.012 0.002; collision box size=0.012 0.012 0.002
- link l_pinky_L2: geometry collision mesh filename=../ability_hand/meshes/collision/idx-F2_C.obj; collision sphere radius=0.007
- link l_ring_L1: geometry collision box size=0.012 0.012 0.002; collision box size=0.012 0.012 0.002
- link l_ring_L2: geometry collision mesh filename=../ability_hand/meshes/collision/idx-F2_C.obj; collision sphere radius=0.007
- link l_thumb_L1: geometry collision mesh filename=../ability_hand/meshes/collision/thumb-F1_C.obj; visual mesh filename=../ability_hand/meshes/visual/thumb-F1.obj
- link l_thumb_L2: geometry collision mesh filename=../ability_hand/meshes/collision/thumb-F2_C.obj; visual mesh filename=../ability_hand/meshes/visual/thumb-F2.obj
- link l_thumb_base: geometry collision mesh filename=../ability_hand/meshes/collision/FB_palm_ref.obj; visual mesh filename=../ability_hand/meshes/visual/FB_palm_ref.obj
- link r_base: geometry collision mesh filename=../ability_hand/meshes/collision/wristmesh_C.obj; visual mesh filename=../ability_hand/meshes/visual/wristmesh.obj
- link r_index_L1: geometry collision box size=0.012 0.012 0.002; collision box size=0.012 0.012 0.002
- link r_index_L2: geometry collision mesh filename=../ability_hand/meshes/collision/idx-F2_C.obj; collision sphere radius=0.007
- link r_middle_L1: geometry collision box size=0.012 0.012 0.002; collision box size=0.012 0.012 0.002
- link r_middle_L2: geometry collision mesh filename=../ability_hand/meshes/collision/idx-F2_C.obj; collision sphere radius=0.007
- link r_pinky_L1: geometry collision box size=0.012 0.012 0.002; collision box size=0.012 0.012 0.002
- link r_pinky_L2: geometry collision mesh filename=../ability_hand/meshes/collision/idx-F2_C.obj; collision sphere radius=0.007
- link r_ring_L1: geometry collision box size=0.012 0.012 0.002; collision box size=0.012 0.012 0.002
- link r_ring_L2: geometry collision mesh filename=../ability_hand/meshes/collision/idx-F2_C.obj; collision sphere radius=0.007
- link r_thumb_L1: geometry collision mesh filename=../ability_hand/meshes/collision/thumb-F1-MIR_C.obj; visual mesh filename=../ability_hand/meshes/visual/thumb-F1-MIR.obj
- link r_thumb_L2: geometry collision mesh filename=../ability_hand/meshes/collision/thumb-F2_C.obj; visual mesh filename=../ability_hand/meshes/visual/thumb-F2.obj
- link r_thumb_base: geometry collision mesh filename=../ability_hand/meshes/collision/FB_palm_ref_MIR.obj; visual mesh filename=../ability_hand/meshes/visual/FB_palm_ref_MIR.obj

File: ace_teleop/assets/xarm7_ability/xarm7_ability_left_hand.urdf (robot description, URDF)
Before this commit: robot xarm7, 25 links, 24 joints
Links:
- link base: geometry collision mesh filename=../ability_hand/meshes/collision/wristmesh_C.obj; visual mesh filename=../ability_hand/meshes/visual/wristmesh.obj
- link index_L1: geometry collision box size=0.012 0.012 0.002; collision box size=0.012 0.012 0.002
- link index_L2: geometry collision mesh filename=../ability_hand/meshes/collision/idx-F2_C.obj; collision sphere radius=0.007
- link link1: geometry collision mesh filename=xarm7/meshes/collision/link1.obj; visual mesh filename=xarm7/meshes/visual/link1.glb
- link link2: geometry collision mesh filename=xarm7/meshes/collision/link2.obj; visual mesh filename=xarm7/meshes/visual/link2.glb
- link link3: geometry collision mesh filename=xarm7/meshes/collision/link3.obj; visual mesh filename=xarm7/meshes/visual/link3.glb
- link link4: geometry collision mesh filename=xarm7/meshes/collision/link4.obj; visual mesh filename=xarm7/meshes/visual/link4.glb
- link link5: geometry collision mesh filename=xarm7/meshes/collision/link5.obj; visual mesh filename=xarm7/meshes/visual/link5.glb
- link link6: geometry collision mesh filename=xarm7/meshes/collision/link6.obj; visual mesh filename=xarm7/meshes/visual/link6.glb
- link link7: geometry collision cylinder length=0.018 radius=0.0365; collision mesh filename=xarm7/meshes/collision/link7.obj
- link link_base: geometry collision mesh filename=xarm7/meshes/collision/link_base.obj; visual mesh filename=xarm7/meshes/visual/link_base.glb
- link middle_L1: geometry collision box size=0.012 0.012 0.002; collision box size=0.012 0.012 0.002
- link middle_L2: geometry collision mesh filename=../ability_hand/meshes/collision/idx-F2_C.obj; collision sphere radius=0.007
- link pinky_L1: geometry collision box size=0.012 0.012 0.002; collision box size=0.012 0.012 0.002
- link pinky_L2: geometry collision mesh filename=../ability_hand/meshes/collision/idx-F2_C.obj; collision sphere radius=0.007
- link ring_L1: geometry collision box size=0.012 0.012 0.002; collision box size=0.012 0.012 0.002
- link ring_L2: geometry collision mesh filename=../ability_hand/meshes/collision/idx-F2_C.obj; collision sphere radius=0.007
- link thumb_L1: geometry collision mesh filename=../ability_hand/meshes/collision/thumb-F1_C.obj; visual mesh filename=../ability_hand/meshes/visual/thumb-F1.obj
- link thumb_L2: geometry collision mesh filename=../ability_hand/meshes/collision/thumb-F2_C.obj; visual mesh filename=../ability_hand/meshes/visual/thumb-F2.obj
- link thumb_base: geometry collision mesh filename=../ability_hand/meshes/collision/FB_palm_ref.obj; visual mesh filename=../ability_hand/meshes/visual/FB_palm_ref.obj

File: ace_teleop/assets/xarm7_ability/xarm7_ability_right_hand.urdf (robot description, URDF)
Before this commit: robot xarm7, 25 links, 24 joints
Links:
- added link ace
- added link ace_1
- link base: geometry collision mesh filename=../ability_hand/meshes/collision/wristmesh_C.obj; visual mesh filename=../ability_hand/meshes/visual/wristmesh.obj
- link index_L1: geometry collision box size=0.012 0.012 0.002; collision box size=0.012 0.012 0.002
- link index_L2: geometry collision mesh filename=../ability_hand/meshes/collision/idx-F2_C.obj; collision sphere radius=0.007
- link link1: geometry collision mesh filename=./xarm7/meshes/collision/link1.obj; visual mesh filename=./xarm7/meshes/visual/link1.glb
- link link2: geometry collision mesh filename=./xarm7/meshes/collision/link2.obj; visual mesh filename=./xarm7/meshes/visual/link2.glb
- link link3: geometry collision mesh filename=./xarm7/meshes/collision/link3.obj; visual mesh filename=./xarm7/meshes/visual/link3.glb
- link link4: geometry collision mesh filename=./xarm7/meshes/collision/link4.obj; visual mesh filename=./xarm7/meshes/visual/link4.glb
- link link5: geometry collision mesh filename=./xarm7/meshes/collision/link5.obj; visual mesh filename=./xarm7/meshes/visual/link5.glb
- link link6: geometry collision mesh filename=./xarm7/meshes/collision/link6.obj; visual mesh filename=./xarm7/meshes/visual/link6.glb
- link link7: geometry collision cylinder length=0.018 radius=0.0365; collision mesh filename=./xarm7/meshes/collision/link7.obj
- link link_base: geometry collision mesh filename=./xarm7/meshes/collision/link_base.obj; visual mesh filename=./xarm7/meshes/visual/link_base.glb
- link middle_L1: geometry collision box size=0.012 0.012 0.002; collision box size=0.012 0.012 0.002
- link middle_L2: geometry collision mesh filename=../ability_hand/meshes/collision/idx-F2_C.obj; collision sphere radius=0.007
- link pinky_L1: geometry collision box size=0.012 0.012 0.002; collision box size=0.012 0.012 0.002
- link pinky_L2: geometry collision mesh filename=../ability_hand/meshes/collision/idx-F2_C.obj; collision sphere radius=0.007
- link ring_L1: geometry collision box size=0.012 0.012 0.002; collision box size=0.012 0.012 0.002
- link ring_L2: geometry collision mesh filename=../ability_hand/meshes/collision/idx-F2_C.obj; collision sphere radius=0.007
- link thumb_L1: geometry collision mesh filename=../ability_hand/meshes/collision/thumb-F1-MIR_C.obj; visual mesh filename=../ability_hand/meshes/visual/thumb-F1-MIR.obj
- link thumb_L2: geometry collision mesh filename=../ability_hand/meshes/collision/thumb-F2_C.obj; visual mesh filename=../ability_hand/meshes/visual/thumb-F2.obj
- link thumb_base: geometry collision mesh filename=../ability_hand/meshes/collision/FB_palm_ref_MIR.obj; visual mesh filename=../ability_hand/meshes/visual/FB_palm_ref_MIR.obj
Joints:
- added joint ace_joint: type fixed, parent base, child ace, origin xyz=0 0 0 rpy=0 -1.57 0
- added joint ace_joint_1: type fixed, parent ace, child ace_1, origin xyz=0 0 0 rpy=0 1.57 0
- joint wrist2thumb: parent base -> ace_1
